File: metropolislefty.kicad_pcb (KiCad board)
At the start: 2 copper layers, 91.3 x 55.6 mm, 26 parts, among them SW1 SW_Push, U1 ATmega32U4-AU, Y1 Crystal_GND24_Small

Commit message: Alpha v0.0.1 Rev 0
Parts:
- added C9: 10nF, Capacitor_SMD:C_0805_2012Metric, F.Cu at (481.0, 164.4)
- added D10: D_Small, Diode_THT:D_DO-35_SOD27_P7.62mm_Horizontal, B.Cu at (100.3, 194.6)
- added D100: D_Small, Diode_THT:D_DO-35_SOD27_P7.62mm_Horizontal, B.Cu at (462.0, 195.3)
- added D101: D_Small, Diode_THT:D_DO-35_SOD27_P7.62mm_Horizontal, B.Cu at (462.0, 214.3)
- added D102: D_Small, Diode_THT:D_DO-35_SOD27_P7.62mm_Horizontal, B.Cu at (462.0, 271.5)
- added D103: D_Small, Diode_THT:D_DO-35_SOD27_P7.62mm_Horizontal, B.Cu at (433.4, 166.7)
- added D104: D_Small, Diode_THT:D_DO-35_SOD27_P7.62mm_Horizontal, B.Cu at (481.0, 195.3)
- added D105: D_Small, Diode_THT:D_DO-35_SOD27_P7.62mm_Horizontal, B.Cu at (481.0, 252.4)
- added D106: D_Small, Diode_THT:D_DO-35_SOD27_P7.62mm_Horizontal, B.Cu at (481.0, 271.5)
- added D107: D_Small, Diode_THT:D_DO-35_SOD27_P7.62mm_Horizontal, B.Cu at (500.1, 195.3)
- added D108: D_Small, Diode_THT:D_DO-35_SOD27_P7.62mm_Horizontal, B.Cu at (500.1, 214.3)
- added D109: D_Small, Diode_THT:D_DO-35_SOD27_P7.62mm_Horizontal, B.Cu at (500.1, 271.5)
- added D11: D_Small, Diode_THT:D_DO-35_SOD27_P7.62mm_Horizontal, B.Cu at (100.0, 214.3)
- added D110: WS2812B, LED_SMD:LED_WS2812B_PLCC4_5.0x5.0mm_P3.2mm, F.Cu at (385.8, 138.1)
- added D111: WS2812B, LED_SMD:LED_WS2812B_PLCC4_5.0x5.0mm_P3.2mm, F.Cu at (404.8, 138.1)
- added D112: WS2812B, LED_SMD:LED_WS2812B_PLCC4_5.0x5.0mm_P3.2mm, F.Cu at (423.9, 138.1)
- added D12: D_Small, Diode_THT:D_DO-35_SOD27_P7.62mm_Horizontal, B.Cu at (100.0, 233.4)
- added D13: D_Small, Diode_THT:D_DO-35_SOD27_P7.62mm_Horizontal, B.Cu at (100.0, 252.4)
- added D14: D_Small, Diode_THT:D_DO-35_SOD27_P7.62mm_Horizontal, B.Cu at (119.1, 166.7)
- added D15: D_Small, Diode_THT:D_DO-35_SOD27_P7.62mm_Horizontal, B.Cu at (119.1, 147.6)
- added D16: D_Small, Diode_THT:D_DO-35_SOD27_P7.62mm_Horizontal, B.Cu at (119.3, 194.3)
- added D17: D_Small, Diode_THT:D_DO-35_SOD27_P7.62mm_Horizontal, B.Cu at (119.1, 219.1)
- added D18: D_Small, Diode_THT:D_DO-35_SOD27_P7.62mm_Horizontal, B.Cu at (119.1, 242.9)
- added D19: D_Small, Diode_THT:D_DO-35_SOD27_P7.62mm_Horizontal, B.Cu at (119.1, 257.2)
- added D20: D_Small, Diode_THT:D_DO-35_SOD27_P7.62mm_Horizontal, B.Cu at (119.1, 271.5)
- added D21: D_Small, Diode_THT:D_DO-35_SOD27_P7.62mm_Horizontal, B.Cu at (138.1, 166.7)
- added D22: D_Small, Diode_THT:D_DO-35_SOD27_P7.62mm_Horizontal, B.Cu at (138.1, 147.6)
- added D23: D_Small, Diode_THT:D_DO-35_SOD27_P7.62mm_Horizontal, B.Cu at (138.1, 195.3)
- added D24: D_Small, Diode_THT:D_DO-35_SOD27_P7.62mm_Horizontal, B.Cu at (139.6, 224.9)
- added D25: D_Small, Diode_THT:D_DO-35_SOD27_P7.62mm_Horizontal, B.Cu at (139.4, 262.5)
- added D26: D_Small, Diode_THT:D_DO-35_SOD27_P7.62mm_Horizontal, B.Cu at (166.7, 166.7)
- added D27: D_Small, Diode_THT:D_DO-35_SOD27_P7.62mm_Horizontal, B.Cu at (166.7, 195.3)
- added D28: D_Small, Diode_THT:D_DO-35_SOD27_P7.62mm_Horizontal, B.Cu at (174.1, 214.3)
- added D29: D_Small, Diode_THT:D_DO-35_SOD27_P7.62mm_Horizontal, B.Cu at (176.2, 233.4)
- added D30: D_Small, Diode_THT:D_DO-35_SOD27_P7.62mm_Horizontal, B.Cu at (190.5, 252.4)
- added D31: D_Small, Diode_THT:D_DO-35_SOD27_P7.62mm_Horizontal, B.Cu at (195.3, 271.5)
- added D32: D_Small, Diode_THT:D_DO-35_SOD27_P7.62mm_Horizontal, B.Cu at (185.7, 166.7)
- added D33: D_Small, Diode_THT:D_DO-35_SOD27_P7.62mm_Horizontal, B.Cu at (185.7, 195.3)
- added D34: D_Small, Diode_THT:D_DO-35_SOD27_P7.62mm_Horizontal, B.Cu at (195.3, 214.3)
- added D35: D_Small, Diode_THT:D_DO-35_SOD27_P7.62mm_Horizontal, B.Cu at (200.0, 233.4)
- added D36: D_Small, Diode_THT:D_DO-35_SOD27_P7.62mm_Horizontal, B.Cu at (209.6, 252.4)
- added D37: D_Small, Diode_THT:D_DO-35_SOD27_P7.62mm_Horizontal, B.Cu at (171.4, 271.5)
- added D38: D_Small, Diode_THT:D_DO-35_SOD27_P7.62mm_Horizontal, B.Cu at (204.8, 166.7)
- added D39: D_Small, Diode_THT:D_DO-35_SOD27_P7.62mm_Horizontal, B.Cu at (204.8, 195.3)
- added D40: D_Small, Diode_THT:D_DO-35_SOD27_P7.62mm_Horizontal, B.Cu at (214.3, 214.3)
- added D41: D_Small, Diode_THT:D_DO-35_SOD27_P7.62mm_Horizontal, B.Cu at (219.1, 233.4)
- added D42: D_Small, Diode_THT:D_DO-35_SOD27_P7.62mm_Horizontal, B.Cu at (228.6, 252.4)
- added D43: D_Small, Diode_THT:D_DO-35_SOD27_P7.62mm_Horizontal, B.Cu at (219.1, 271.5)
- added D44: D_Small, Diode_THT:D_DO-35_SOD27_P7.62mm_Horizontal, B.Cu at (223.8, 166.7)
- added D45: D_Small, Diode_THT:D_DO-35_SOD27_P7.62mm_Horizontal, B.Cu at (223.8, 195.3)
- added D46: D_Small, Diode_THT:D_DO-35_SOD27_P7.62mm_Horizontal, B.Cu at (233.4, 214.3)
- added D47: D_Small, Diode_THT:D_DO-35_SOD27_P7.62mm_Horizontal, B.Cu at (238.1, 233.4)
- added D48: D_Small, Diode_THT:D_DO-35_SOD27_P7.62mm_Horizontal, B.Cu at (247.7, 252.4)
- added D49: D_Small, Diode_THT:D_DO-35_SOD27_P7.62mm_Horizontal, B.Cu at (338.1, 271.5)
- added D5: D_Small, Diode_THT:D_DO-35_SOD27_P7.62mm_Horizontal, B.Cu at (81.0, 233.4)
- added D50: D_Small, Diode_THT:D_DO-35_SOD27_P7.62mm_Horizontal, B.Cu at (242.9, 166.7)
- added D51: D_Small, Diode_THT:D_DO-35_SOD27_P7.62mm_Horizontal, B.Cu at (242.9, 195.3)
- added D52: D_Small, Diode_THT:D_DO-35_SOD27_P7.62mm_Horizontal, B.Cu at (252.4, 214.3)
- added D53: D_Small, Diode_THT:D_DO-35_SOD27_P7.62mm_Horizontal, B.Cu at (257.2, 233.4)
- added D54: D_Small, Diode_THT:D_DO-35_SOD27_P7.62mm_Horizontal, B.Cu at (266.7, 252.4)
- added D55: D_Small, Diode_THT:D_DO-35_SOD27_P7.62mm_Horizontal, B.Cu at (361.9, 271.5)
- added D56: D_Small, Diode_THT:D_DO-35_SOD27_P7.62mm_Horizontal, B.Cu at (290.5, 166.7)
- added D57: D_Small, Diode_THT:D_DO-35_SOD27_P7.62mm_Horizontal, B.Cu at (261.9, 195.3)
- added D58: D_Small, Diode_THT:D_DO-35_SOD27_P7.62mm_Horizontal, B.Cu at (271.5, 214.3)
- added D59: D_Small, Diode_THT:D_DO-35_SOD27_P7.62mm_Horizontal, B.Cu at (276.2, 233.4)
- added D6: D_Small, Diode_THT:D_DO-35_SOD27_P7.62mm_Horizontal, B.Cu at (81.0, 252.4)
- added D60: D_Small, Diode_THT:D_DO-35_SOD27_P7.62mm_Horizontal, B.Cu at (285.8, 252.4)
- added D61: D_Small, Diode_THT:D_DO-35_SOD27_P7.62mm_Horizontal, B.Cu at (385.8, 271.5)
- added D62: D_Small, Diode_THT:D_DO-35_SOD27_P7.62mm_Horizontal, B.Cu at (309.6, 166.7)
- added D63: D_Small, Diode_THT:D_DO-35_SOD27_P7.62mm_Horizontal, B.Cu at (281.0, 195.3)
- added D64: D_Small, Diode_THT:D_DO-35_SOD27_P7.62mm_Horizontal, B.Cu at (290.5, 214.3)
- added D65: D_Small, Diode_THT:D_DO-35_SOD27_P7.62mm_Horizontal, B.Cu at (295.3, 233.4)
- added D66: D_Small, Diode_THT:D_DO-35_SOD27_P7.62mm_Horizontal, B.Cu at (304.8, 252.4)
- added D67: D_Small, Diode_THT:D_DO-35_SOD27_P7.62mm_Horizontal, B.Cu at (409.6, 271.5)
- added D68: D_Small, Diode_THT:D_DO-35_SOD27_P7.62mm_Horizontal, B.Cu at (328.6, 166.7)
- added D69: D_Small, Diode_THT:D_DO-35_SOD27_P7.62mm_Horizontal, B.Cu at (300.0, 195.3)
- added D7: D_Small, Diode_THT:D_DO-35_SOD27_P7.62mm_Horizontal, B.Cu at (100.0, 271.5)
- added D70: D_Small, Diode_THT:D_DO-35_SOD27_P7.62mm_Horizontal, B.Cu at (309.6, 214.3)
- added D71: D_Small, Diode_THT:D_DO-35_SOD27_P7.62mm_Horizontal, B.Cu at (314.3, 233.4)
- added D72: D_Small, Diode_THT:D_DO-35_SOD27_P7.62mm_Horizontal, B.Cu at (323.9, 252.4)
- added D73: D_Small, Diode_THT:D_DO-35_SOD27_P7.62mm_Horizontal, B.Cu at (433.4, 271.5)
- added D74: D_Small, Diode_THT:D_DO-35_SOD27_P7.62mm_Horizontal, B.Cu at (347.7, 166.7)
- added D75: D_Small, Diode_THT:D_DO-35_SOD27_P7.62mm_Horizontal, B.Cu at (319.1, 195.3)
- added D76: D_Small, Diode_THT:D_DO-35_SOD27_P7.62mm_Horizontal, B.Cu at (328.6, 214.3)
- added D77: D_Small, Diode_THT:D_DO-35_SOD27_P7.62mm_Horizontal, B.Cu at (333.4, 233.4)
- added D78: D_Small, Diode_THT:D_DO-35_SOD27_P7.62mm_Horizontal, B.Cu at (342.9, 252.4)
- added D79: D_Small, Diode_THT:D_DO-35_SOD27_P7.62mm_Horizontal, B.Cu at (376.2, 166.7)
- added D8: D_Small, Diode_THT:D_DO-35_SOD27_P7.62mm_Horizontal, B.Cu at (100.0, 166.7)
- added D80: D_Small, Diode_THT:D_DO-35_SOD27_P7.62mm_Horizontal, B.Cu at (338.1, 195.3)
- added D81: D_Small, Diode_THT:D_DO-35_SOD27_P7.62mm_Horizontal, B.Cu at (347.7, 214.3)
- added D82: D_Small, Diode_THT:D_DO-35_SOD27_P7.62mm_Horizontal, B.Cu at (352.4, 233.4)
- added D83: D_Small, Diode_THT:D_DO-35_SOD27_P7.62mm_Horizontal, B.Cu at (361.9, 252.4)
- added D84: D_Small, Diode_THT:D_DO-35_SOD27_P7.62mm_Horizontal, B.Cu at (395.3, 166.7)
- added D85: D_Small, Diode_THT:D_DO-35_SOD27_P7.62mm_Horizontal, B.Cu at (357.2, 195.3)
- added D86: D_Small, Diode_THT:D_DO-35_SOD27_P7.62mm_Horizontal, B.Cu at (366.7, 214.3)
- added D87: D_Small, Diode_THT:D_DO-35_SOD27_P7.62mm_Horizontal, B.Cu at (371.5, 233.4)
- added D88: D_Small, Diode_THT:D_DO-35_SOD27_P7.62mm_Horizontal, B.Cu at (381.0, 252.4)
- added D89: D_Small, Diode_THT:D_DO-35_SOD27_P7.62mm_Horizontal, B.Cu at (414.3, 166.7)
- added D9: D_Small, Diode_THT:D_DO-35_SOD27_P7.62mm_Horizontal, B.Cu at (100.1, 147.6)
- added D90: D_Small, Diode_THT:D_DO-35_SOD27_P7.62mm_Horizontal, B.Cu at (376.2, 195.3)
- added D91: D_Small, Diode_THT:D_DO-35_SOD27_P7.62mm_Horizontal, B.Cu at (385.8, 214.3)
- added D92: D_Small, Diode_THT:D_DO-35_SOD27_P7.62mm_Horizontal, B.Cu at (390.5, 233.4)
- added D93: D_Small, Diode_THT:D_DO-35_SOD27_P7.62mm_Horizontal, B.Cu at (433.4, 252.4)
- added D94: D_Small, Diode_THT:D_DO-35_SOD27_P7.62mm_Horizontal, B.Cu at (481.0, 214.3)
- added D95: D_Small, Diode_THT:D_DO-35_SOD27_P7.62mm_Horizontal, B.Cu at (395.3, 195.3)
- added D96: D_Small, Diode_THT:D_DO-35_SOD27_P7.62mm_Horizontal, B.Cu at (406.0, 214.3)
- added D97: D_Small, Diode_THT:D_DO-35_SOD27_P7.62mm_Horizontal, B.Cu at (433.4, 233.4)
- added D98: D_Small, Diode_THT:D_DO-35_SOD27_P7.62mm_Horizontal, B.Cu at (433.4, 195.3)
- added D99: D_Small, Diode_THT:D_DO-35_SOD27_P7.62mm_Horizontal, B.Cu at (433.4, 214.3)
- added MX10: Num_Multiply, MX_Alps_Hybrid:MX-1U, F.Cu at (90.5, 190.5)
- added MX100: Insert, MX_Alps_Hybrid:MX-1U, F.Cu at (452.4, 190.5)
- added MX101: Delete, MX_Alps_Hybrid:MX-1U, F.Cu at (452.4, 209.6)
- added MX102: ArrowLeft, MX_Alps_Hybrid:MX-1U, F.Cu at (452.4, 266.7)
- added MX103: Home, MX_Alps_Hybrid:MX-1U, F.Cu at (471.5, 190.5)
- added MX104: End, MX_Alps_Hybrid:MX-1U, F.Cu at (471.5, 209.6)
- added MX105: ArrowUp, MX_Alps_Hybrid:MX-1U, F.Cu at (471.5, 247.7)
- added MX106: ArrowDown, MX_Alps_Hybrid:MX-1U, F.Cu at (471.5, 266.7)
- added MX107: PageUp, MX_Alps_Hybrid:MX-1U, F.Cu at (490.5, 190.5)
- added MX108: PageDown, MX_Alps_Hybrid:MX-1U, F.Cu at (490.5, 209.6)
- added MX109: ArrowRight, MX_Alps_Hybrid:MX-1U, F.Cu at (490.5, 266.7)
- added MX11: Num_8, MX_Alps_Hybrid:MX-1U, F.Cu at (90.5, 209.6)
- added MX12: Num_5, MX_Alps_Hybrid:MX-1U, F.Cu at (90.5, 228.6)
- added MX13: Num_2, MX_Alps_Hybrid:MX-1U, F.Cu at (90.5, 247.7)
- added MX14: Macro_3, MX_Alps_Hybrid:MX-1U, F.Cu at (109.5, 161.9)
- added MX15: Macro_7, MX_Alps_Hybrid:MX-1U, F.Cu at (109.5, 142.9)
- added MX16: Num_Minus, MX_Alps_Hybrid:MX-1U, F.Cu at (109.5, 190.5)
- added MX17: Num_9, MX_Alps_Hybrid:MX-1U, F.Cu at (109.5, 209.6)
- added MX18: Num_6, MX_Alps_Hybrid:MX-1U, F.Cu at (109.5, 228.6)
- added MX19: Num_3, MX_Alps_Hybrid:MX-1U, F.Cu at (109.5, 247.7)
- added MX20: Num_., MX_Alps_Hybrid:MX-1U, F.Cu at (109.5, 266.7)
- added MX21: Macro_4, MX_Alps_Hybrid:MX-1U, F.Cu at (128.6, 161.9)
- added MX22: Macro_8, MX_Alps_Hybrid:MX-1U, F.Cu at (128.6, 142.9)
- added MX23: Num_Delete, MX_Alps_Hybrid:MX-1U, F.Cu at (128.6, 190.5)
- added MX24: Num_Plus, MX_Alps_Hybrid:MX-2U, F.Cu at (128.6, 219.1)
- added MX25: Num_Return, MX_Alps_Hybrid:MX-2U, F.Cu at (128.6, 257.2)
- added MX26: Escape, MX_Alps_Hybrid:MX-1U, F.Cu at (157.2, 161.9)
- added MX27: `, MX_Alps_Hybrid:MX-1U, F.Cu at (157.2, 190.5)
- added MX28: Tab, MX_Alps_Hybrid:MX-1.5U, F.Cu at (161.9, 209.6)
- added MX29: Caps Lock, MX_Alps_Hybrid:MX-1.75U, F.Cu at (164.3, 228.6)
- added MX30: Shift_Left, MX_Alps_Hybrid:MX-2.25U, F.Cu at (169.1, 247.7)
- added MX31: Control_Left, MX_Alps_Hybrid:MX-1.25U, F.Cu at (183.4, 266.7)
- added MX32: F1, MX_Alps_Hybrid:MX-1U, F.Cu at (195.3, 161.9)
- added MX33: 1, MX_Alps_Hybrid:MX-1U, F.Cu at (176.2, 190.5)
- added MX34: Q, MX_Alps_Hybrid:MX-1U, F.Cu at (185.7, 209.6)
- added MX35: A, MX_Alps_Hybrid:MX-1U, F.Cu at (190.5, 228.6)
- added MX36: Z, MX_Alps_Hybrid:MX-1U, F.Cu at (200.0, 247.7)
- added MX37: Code_Left, MX_Alps_Hybrid:MX-1.25U, F.Cu at (159.5, 266.7)
- added MX38: F2, MX_Alps_Hybrid:MX-1U, F.Cu at (214.3, 161.9)
- added MX39: 2, MX_Alps_Hybrid:MX-1U, F.Cu at (195.3, 190.5)
- added MX40: W, MX_Alps_Hybrid:MX-1U, F.Cu at (204.8, 209.6)
- added MX41: S, MX_Alps_Hybrid:MX-1U, F.Cu at (209.6, 228.6)
- added MX42: X, MX_Alps_Hybrid:MX-1U, F.Cu at (219.1, 247.7)
- added MX43: Alt_Left, MX_Alps_Hybrid:MX-1.25U, F.Cu at (207.2, 266.7)
- added MX44: F3, MX_Alps_Hybrid:MX-1U, F.Cu at (233.4, 161.9)
- added MX45: 3, MX_Alps_Hybrid:MX-1U, F.Cu at (214.3, 190.5)
- added MX46: E, MX_Alps_Hybrid:MX-1U, F.Cu at (223.8, 209.6)
- added MX47: D, MX_Alps_Hybrid:MX-1U, F.Cu at (228.6, 228.6)
- added MX48: C, MX_Alps_Hybrid:MX-1U, F.Cu at (238.1, 247.7)
- added MX49: Space, MX_Alps_Hybrid:MX-6.25U, F.Cu at (278.6, 266.7)
- added MX5: Num_4, MX_Alps_Hybrid:MX-1U, F.Cu at (71.4, 228.6)
- added MX50: F4, MX_Alps_Hybrid:MX-1U, F.Cu at (252.4, 161.9)
- added MX51: 4, MX_Alps_Hybrid:MX-1U, F.Cu at (233.4, 190.5)
- added MX52: R, MX_Alps_Hybrid:MX-1U, F.Cu at (242.9, 209.6)
- added MX53: F, MX_Alps_Hybrid:MX-1U, F.Cu at (247.7, 228.6)
- added MX54: V, MX_Alps_Hybrid:MX-1U, F.Cu at (257.2, 247.7)
- added MX55: Super, MX_Alps_Hybrid:MX-1.25U, F.Cu at (350.0, 266.7)
- added MX56: F5, MX_Alps_Hybrid:MX-1U, F.Cu at (281.0, 161.9)
- added MX57: 5, MX_Alps_Hybrid:MX-1U, F.Cu at (252.4, 190.5)
- added MX58: T, MX_Alps_Hybrid:MX-1U, F.Cu at (261.9, 209.6)
- added MX59: G, MX_Alps_Hybrid:MX-1U, F.Cu at (266.7, 228.6)
- added MX6: Num_1, MX_Alps_Hybrid:MX-1U, F.Cu at (71.4, 247.7)
- added MX60: B, MX_Alps_Hybrid:MX-1U, F.Cu at (276.2, 247.7)
- added MX61: Alt_Right, MX_Alps_Hybrid:MX-1.25U, F.Cu at (373.9, 266.7)
- added MX62: F6, MX_Alps_Hybrid:MX-1U, F.Cu at (300.0, 161.9)
- added MX63: 6, MX_Alps_Hybrid:MX-1U, F.Cu at (271.5, 190.5)
- added MX64: Y, MX_Alps_Hybrid:MX-1U, F.Cu at (281.0, 209.6)
- added MX65: H, MX_Alps_Hybrid:MX-1U, F.Cu at (285.8, 228.6)
- added MX66: N, MX_Alps_Hybrid:MX-1U, F.Cu at (295.3, 247.7)
- added MX67: Code_Right, MX_Alps_Hybrid:MX-1.25U, F.Cu at (397.7, 266.7)
- added MX68: F7, MX_Alps_Hybrid:MX-1U, F.Cu at (319.1, 161.9)
- added MX69: 7, MX_Alps_Hybrid:MX-1U, F.Cu at (290.5, 190.5)
- added MX7: Num_0, MX_Alps_Hybrid:MX-2U, F.Cu at (81.0, 266.7)
- added MX70: U, MX_Alps_Hybrid:MX-1U, F.Cu at (300.0, 209.6)
- added MX71: J, MX_Alps_Hybrid:MX-1U, F.Cu at (304.8, 228.6)
- added MX72: M, MX_Alps_Hybrid:MX-1U, F.Cu at (314.3, 247.7)
- added MX73: Control_Right, MX_Alps_Hybrid:MX-1.25U, F.Cu at (421.5, 266.7)
- added MX74: F8, MX_Alps_Hybrid:MX-1U, F.Cu at (338.1, 161.9)
- added MX75: 8, MX_Alps_Hybrid:MX-1U, F.Cu at (309.6, 190.5)
- added MX76: I, MX_Alps_Hybrid:MX-1U, F.Cu at (319.1, 209.6)
- added MX77: K, MX_Alps_Hybrid:MX-1U, F.Cu at (323.9, 228.6)
- added MX78: ,, MX_Alps_Hybrid:MX-1U, F.Cu at (333.4, 247.7)
- added MX79: F9, MX_Alps_Hybrid:MX-1U, F.Cu at (366.7, 161.9)
- added MX8: Macro_2, MX_Alps_Hybrid:MX-1U, F.Cu at (90.5, 161.9)
- added MX80: 9, MX_Alps_Hybrid:MX-1U, F.Cu at (328.6, 190.5)
- added MX81: O, MX_Alps_Hybrid:MX-1U, F.Cu at (338.1, 209.6)
- added MX82: L, MX_Alps_Hybrid:MX-1U, F.Cu at (342.9, 228.6)
- added MX83: ., MX_Alps_Hybrid:MX-1U, F.Cu at (352.4, 247.7)
- added MX84: F10, MX_Alps_Hybrid:MX-1U, F.Cu at (385.8, 161.9)
- added MX85: 0, MX_Alps_Hybrid:MX-1U, F.Cu at (347.7, 190.5)
- added MX86: P, MX_Alps_Hybrid:MX-1U, F.Cu at (357.2, 209.6)
- added MX87: ;, MX_Alps_Hybrid:MX-1U, F.Cu at (361.9, 228.6)
- added MX88: /, MX_Alps_Hybrid:MX-1U, F.Cu at (371.5, 247.7)
- added MX89: F11, MX_Alps_Hybrid:MX-1U, F.Cu at (404.8, 161.9)
- added MX9: Macro_6, MX_Alps_Hybrid:MX-1U, F.Cu at (90.5, 142.9)
- added MX90: -, MX_Alps_Hybrid:MX-1U, F.Cu at (366.7, 190.5)
- added MX91: [, MX_Alps_Hybrid:MX-1U, F.Cu at (376.2, 209.6)
- added MX92: ', MX_Alps_Hybrid:MX-1U, F.Cu at (381.0, 228.6)
- added MX93: Shift, MX_Alps_Hybrid:MX-2.75U, F.Cu at (407.2, 247.7)
- added MX94: F12, MX_Alps_Hybrid:MX-1U, F.Cu at (423.9, 161.9)
- added MX95: =, MX_Alps_Hybrid:MX-1U, F.Cu at (385.8, 190.5)
- added MX96: ], MX_Alps_Hybrid:MX-1U, F.Cu at (395.3, 209.6)
- added MX97: Return, MX_Alps_Hybrid:MX-2.25U, F.Cu at (412.0, 228.6)
- added MX98: Backspace, MX_Alps_Hybrid:MX-2U, F.Cu at (414.3, 190.5)
- added MX99: \, MX_Alps_Hybrid:MX-1.5U, F.Cu at (419.1, 209.6)
- added R6: 300, Resistor_SMD:R_0805_2012Metric, F.Cu at (376.2, 138.1)
- added R7: 33K, Resistor_SMD:R_0805_2012Metric, F.Cu at (448.6, 167.0)
- added R8: 15k, Resistor_SMD:R_0805_2012Metric, F.Cu at (447.7, 152.4)
- added R9: 15k, Resistor_SMD:R_0805_2012Metric, F.Cu at (481.0, 152.4)
- added REF**: MountingHole_2.5mm_Pad_Via, MountingHole:MountingHole_2.5mm_Pad_Via, F.Cu at (500.1, 133.3)
- added REF**: MountingHole_2.5mm_Pad_Via, MountingHole:MountingHole_2.5mm_Pad_Via, F.Cu at (500.1, 276.2)
- added REF**: MountingHole_2.5mm_Pad_Via, MountingHole:MountingHole_2.5mm_Pad_Via, F.Cu at (61.9, 276.2)
- added REF**: MountingHole_2.5mm_Pad_Via, MountingHole:MountingHole_2.5mm_Pad_Via, F.Cu at (61.9, 133.3)
- added SW2: Rotary_Encoder_Switch, Rotary_Encoder:RotaryEncoder_Alps_EC11E-Switch_Vertical_H20mm, F.Cu at (455.0, 156.3)
- D1, D2, D3, D4: footprint Diode_SMD:D_SOD-123 -> Diode_THT:D_DO-35_SOD27_P7.62mm_Horizontal
- MX1: value MX-NoLED -> Macro_1
- MX2: value MX-NoLED -> Macro_5
- MX3: value MX-NoLED -> Num_Divide
- MX4: value MX-NoLED -> Num_7
- moved C2 222.6 mm to (267.2, 166.4), turned to 180 degrees
- moved C1 221.7 mm to (288.1, 140.1), turned to 270 degrees
- moved USB1 220.2 mm to (278.6, 130.0)
- moved R2 218.1 mm to (280.5, 146.5)
- moved R3 217.5 mm to (277.5, 146.4)
- moved C4 214.7 mm to (288.1, 144.8), turned to 90 degrees
- moved C8 212.4 mm to (277.6, 152.0), turned to 90 degrees
- moved C7 210.7 mm to (292.9, 144.8), turned to 270 degrees
- moved F1 209.5 mm to (259.9, 138.4)
- moved C3 208.8 mm to (265.0, 138.7)
- moved Y1 205.7 mm to (288.1, 149.6)
- moved U1 200.9 mm to (267.3, 150.3), turned to 180 degrees
- moved C5 197.1 mm to (252.5, 154.1), turned to 270 degrees
- moved C6 188.3 mm to (262.5, 160.9), turned to 0 degrees
- moved R5 186.5 mm to (247.1, 154.1), turned to 90 degrees
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Connections:
- D1 pad 1: ROW0 -> ROW1
- D3 pad 1: ROW1 -> ROW2
- D4 pad 1: ROW1 -> ROW3
- MX2 pad 1: COL1 -> COL3
- MX4 pad 1: COL1 -> COL0
- R5 pad 2: Net-(R5-Pad2) -> COL1
- U1 pad 1: Net-(U1-Pad1) -> COL13
- U1 pad 10: Net-(U1-Pad10) -> ROW1
- U1 pad 11: Net-(U1-Pad11) -> ROW3
- U1 pad 12: Net-(U1-Pad12) -> COL12
- U1 pad 18: Net-(U1-Pad18) -> ROW2
- U1 pad 19: ROW0 -> COL9
- U1 pad 20: COL1 -> COL8
- U1 pad 21: COL0 -> ROW0
- U1 pad 22: ROW1 -> COL10
- U1 pad 25: Net-(U1-Pad25) -> COL7
- U1 pad 26: Net-(U1-Pad26) -> COL6
- U1 pad 27: Net-(U1-Pad27) -> COL11
- U1 pad 28: Net-(U1-Pad28) -> COL5
- U1 pad 29: Net-(U1-Pad29) -> COL4
- U1 pad 30: Net-(U1-Pad30) -> COL0
- U1 pad 31: Net-(U1-Pad31) -> COL3
- U1 pad 32: Net-(U1-Pad32) -> COL2
- U1 pad 33: Net-(R5-Pad2) -> COL1
- U1 pad 36: Net-(U1-Pad36) -> STATUS_LEDS
- U1 pad 37: Net-(U1-Pad37) -> COL18
- U1 pad 38: Net-(U1-Pad38) -> COL17
- U1 pad 39: Net-(U1-Pad39) -> COL14
- U1 pad 40: Net-(U1-Pad40) -> COL15
- U1 pad 41: Net-(U1-Pad41) -> COL16
- U1 pad 42: Net-(U1-Pad42) -> ENCODER
- U1 pad 8: Net-(U1-Pad8) -> ROW5
- U1 pad 9: Net-(U1-Pad9) -> ROW4
Routing:
- net ROW4: track 0.00 -> 661.1 mm, vias 0 -> 10
- net ROW5: track 0.00 -> 587.1 mm, vias 0 -> 6
- net ROW3: track 0.00 -> 577.2 mm, vias 0 -> 6
- net ROW2: track 0.00 -> 538.5 mm, vias 0 -> 8
- net ROW1: track 63.4 -> 509.8 mm, vias 2 -> 5
- net COL3: track 0.00 -> 398.4 mm, vias 0 -> 4
- net COL4: track 0.00 -> 386.6 mm, vias 0 -> 4
- net COL5: track 0.00 -> 378.1 mm, vias 0 -> 6
- net ROW0: track 62.3 -> 433.9 mm
- net COL7: track 0.00 -> 316.0 mm, vias 0 -> 9
- net COL17: track 0.00 -> 313.4 mm, vias 0 -> 3
- net COL6: track 0.00 -> 303.1 mm, vias 0 -> 4
- net COL2: track 0.00 -> 290.0 mm, vias 0 -> 2
- net COL18: track 0.00 -> 277.8 mm, vias 0 -> 4
- net COL16: track 0.00 -> 273.4 mm, vias 0 -> 1
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- added copper zone on B.Cu, net GND
Other:
- board size 91.3 x 55.6 mm -> 449 x 153 mm
- board text added: "Kasper Southpaw V1.0 Rev 0 01/2020"
