File: metropolislefty.kicad_pcb (KiCad board)
At the start: 2 copper layers, 91.3 x 55.6 mm, 26 parts, among them SW1 SW_Push, U1 ATmega32U4-AU, Y1 Crystal_GND24_Small

Commit message: Revision 1 Test w/ USB C
Parts:
- added D5: WS2812B, LED_SMD:LED_WS2812B_PLCC4_5.0x5.0mm_P3.2mm, F.Cu at (59.5, 91.3)
- added D6: WS2812B, LED_SMD:LED_WS2812B_PLCC4_5.0x5.0mm_P3.2mm, F.Cu at (59.5, 100.0)
- added D7: WS2812B, LED_SMD:LED_WS2812B_PLCC4_5.0x5.0mm_P3.2mm, F.Cu at (59.5, 110.3)
- added R10: 33k, Resistor_SMD:R_0805_2012Metric, B.Cu at (67.5, 119.1)
- added R6: 5k1, Resistor_SMD:R_0805_2012Metric, B.Cu at (85.7, 86.5)
- added R7: 470, Resistor_SMD:R_0805_2012Metric, F.Cu at (59.5, 84.9)
- added R8: 15k, Resistor_SMD:R_0805_2012Metric, B.Cu at (85.7, 110.3)
- added R9: 15k, Resistor_SMD:R_0805_2012Metric, B.Cu at (73.0, 107.2)
- added SW2: Rotary_Encoder_Switch, Rotary_Encoder:RotaryEncoder_Alps_EC11E-Switch_Vertical_H20mm, F.Cu at (73.0, 115.9)
- C1: value 4.7nF -> 10nF
- D1, D2, D3, D4: footprint Diode_SMD:D_SOD-123 -> Diode_THT:D_DO-35_SOD27_P7.62mm_Horizontal; moved to F.Cu
- R1: value 1M -> 5k1
- USB1: value Molex-0548190589 -> HRO-TYPE-C-31-M-12; footprint random-keyboard-parts:Molex-0548190589 -> Type-C:HRO-TYPE-C-31-M-12
- moved D2 42.0 mm to (95.2, 81.8)
- moved D4 41.1 mm to (96.0, 115.1), turned to 270 degrees
- moved C1 35.2 mm to (88.9, 110.3), turned to 90 degrees
- moved C2 34.2 mm to (91.8, 95.2)
- moved D1 27.4 mm to (91.3, 81.8)
- moved D3 26.4 mm to (92.1, 115.1), turned to 270 degrees
- moved C3 15.4 mm to (70.6, 103.2), turned to 90 degrees
- moved C5 15.2 mm to (73.8, 94.5), turned to 270 degrees
- moved USB1 15.2 mm to (81.0, 71.4), turned to 0 degrees
- moved R2 11.9 mm to (82.5, 86.5)
- moved F1 11.7 mm to (69.2, 85.7), turned to 180 degrees
- moved C8 11.1 mm to (85.7, 90.5)
- moved R3 11.1 mm to (79.4, 86.5)
- moved R4 10.4 mm to (88.9, 86.5), turned to 270 degrees
- moved C6 10.3 mm to (94.5, 102.4), turned to 0 degrees
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Connections:
- C1 pad 1: Net-(C1-Pad1) -> ENC
- F1 pad 1: VCC -> VBUS
- R1 pad 1: Net-(C1-Pad1) -> GND
- R1 pad 2: GND -> Net-(R1-Pad2)
- U1 pad 1: Net-(U1-Pad1) -> LEDS
- U1 pad 11: Net-(U1-Pad11) -> ROW0
- U1 pad 19: ROW0 -> Net-(U1-Pad19)
- U1 pad 42: Net-(U1-Pad42) -> ENC
- USB1 pad 2: Net-(USB1-Pad2) -> VBUS
- USB1 pad 3: D+ -> Net-(USB1-Pad3)
- USB1 pad 4: D- -> Net-(R1-Pad2)
- USB1 pad 5: VCC -> D-
- USB1 pad 6: Net-(C1-Pad1) -> D+
Routing:
- net +5V: track 105.1 -> 174.0 mm, vias 7 -> 11
- net ENC: track 0.00 -> 55.3 mm, vias 0 -> 2
- net ROW1: track 63.4 -> 16.4 mm
- net Net-(D4-Pad2): track 7.08 -> 52.4 mm
- net ROW0: track 62.3 -> 19.0 mm, vias 2 -> 1
- net Net-(D2-Pad2): track 7.41 -> 40.7 mm
- net Net-(D3-Pad2): track 7.08 -> 36.0 mm
- net Net-(C1-Pad1): track 28.6 -> 0.00 mm
- net LEDS: track 0.00 -> 22.4 mm, vias 0 -> 1
- net VBUS: track 0.00 -> 18.4 mm
- net Net-(D1-Pad2): track 7.41 -> 24.0 mm
- net Net-(C7-Pad2): track 19.1 -> 7.48 mm, vias 2 -> 0
- net Net-(D6-Pad2): track 0.00 -> 9.74 mm
- net VCC: track 8.72 -> 0.00 mm
- net Net-(D5-Pad2): track 0.00 -> 8.15 mm
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- added copper zone on B.Cu, net GND
Other:
- outline, holes or cut-outs redrawn
- board text added: "Kevin Kasper Who is he? Numpad Test v02"
