File: metropolislefty.sch (KiCad schematic (older format))
At the start: 15 parts

Commit message: Created test board.
Parts:
- added C1: 4.7nF, Capacitor_SMD:C_0805_2012Metric, symbol Device:C_Small
- added D1, D2, D3, D4: D_Small, Diode_SMD:D_SOD-123, symbol Device:D_Small
- added F1: 500mA, Fuse:Fuse_1206_3216Metric, symbol Device:Polyfuse_Small
- added MX1, MX2, MX3, MX4: MX-NoLED, MX_Alps_Hybrid:MX-1U, symbol MX_Alps_Hybrid:MX-NoLED
- added R1: 1M, Resistor_SMD:R_0805_2012Metric, symbol Device:R_Small
- C2, C3, C4, C5, C6, C7, C8: renamed from C?; footprint (none) -> Capacitor_SMD:C_0805_2012Metric
- R2, R3, R4, R5: renamed from R?; footprint (none) -> Resistor_SMD:R_0805_2012Metric
- SW1: renamed from SW?; footprint (none) -> random-keyboard-parts:SKQG-1155865
- USB1: renamed from USB?; footprint (none) -> random-keyboard-parts:Molex-0548190589
- Y1: renamed from Y?; footprint (none) -> Crystal:Crystal_SMD_3225-4Pin_3.2x2.5mm
- gave numbers to parts that had none: 1
Connections:
- net +5V: now also F1.2; no longer USB1.5 (VBUS)
- net D+: now also USB1.3 (D+)
- net D-: now also USB1.4 (D-)
- net GND: now also USB1.1 (GND), C1.2, R1.2
- net ROW0: now reaches U1.19 (PD1)
- net ROW0: now also D1.1 (K), D2.1 (K)
- net COL1: now reaches U1.20 (PD2)
- net COL1: now also MX2.1 (COL), MX4.1 (COL)
- net COL0: now reaches U1.21 (PD3)
- net COL0: now also MX1.1 (COL), MX3.1 (COL)
- net ROW1: now reaches U1.22 (PD5)
- net ROW1: now also D3.1 (K), D4.1 (K)
- net at USB1.6 (SHIELD): now also C1.1, R1.1
- new net: D1.2 (A), MX1.2 (ROW)
- new net: D3.2 (A), MX3.2 (ROW)
- new net: D2.2 (A), MX2.2 (ROW)
- new net: D4.2 (A), MX4.2 (ROW)
- new net VCC: F1.1, USB1.5 (VBUS)
Other:
- moved on the sheet: C2, C3, C4, C5, C6, C7, C8, R2, R3, R4, R5, SW1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

Commit message: Alpha v0.0.1 Rev 0
Parts:
- removed D1, D2, D3, D4: D_Small, Diode_SMD:D_SOD-123, symbol Device:D_Small
- removed MX1, MX2, MX3, MX4: MX-NoLED, MX_Alps_Hybrid:MX-1U, symbol MX_Alps_Hybrid:MX-NoLED
- added C9: 10nF, Capacitor_SMD:C_0805_2012Metric, symbol Device:C_Small
- added D110, D111, D112: WS2812B, LED_SMD:LED_WS2812B_PLCC4_5.0x5.0mm_P3.2mm, symbol LED:WS2812B
- added R6: 300, Resistor_SMD:R_0805_2012Metric, symbol Device:R_Small
- added R7: 33K, Resistor_SMD:R_0805_2012Metric, symbol Device:R_Small
- added R8, R9: 15k, Resistor_SMD:R_0805_2012Metric, symbol Device:R_Small
- added SW2: Rotary_Encoder_Switch, Rotary_Encoder:RotaryEncoder_Alps_EC11E-Switch_Vertical_H20mm, symbol Device:Rotary_Encoder_Switch
- USB1: symbol random-keyboard-parts:Molex-0548190589 -> metropolislefty-rescue:Molex-0548190589-random-keyboard-parts
Connections:
- net +5V: now also D110.1 (VDD), D111.1 (VDD), D112.1 (VDD), R9.2
- net COL0: now also U1.30 (PB6); no longer U1.21 (PD3)
- net COL1: now also R5.2, U1.33 (~HWB~/PE2); no longer U1.20 (PD2)
- net GND: now also C9.2, D110.3 (VSS), D111.3 (VSS), D112.3 (VSS), SW2.C, SW2.S2
- net ROW0: now also U1.21 (PD3); no longer U1.19 (PD1)
- net ROW1: now also U1.10 (PB2); no longer U1.22 (PD5)
- net COL13: now reaches U1.1 (PE6)
- net ROW3: now reaches U1.11 (PB3)
- net COL12: now reaches U1.12 (PB7)
- net ROW2: now reaches U1.18 (PD0)
- net COL7: now reaches U1.25 (PD4)
- net COL6: now reaches U1.26 (PD6)
- net COL11: now reaches U1.27 (PD7)
- net COL5: now reaches U1.28 (PB4)
- net COL4: now reaches U1.29 (PB5)
- net COL3: now reaches U1.31 (PC6)
- net COL2: now reaches U1.32 (PC7)
- net STATUS_LEDS: now reaches U1.36 (PF7)
- net STATUS_LEDS: now also R6.2
- net COL18: now reaches U1.37 (PF6)
- net COL17: now reaches U1.38 (PF5)
- net COL14: now reaches U1.39 (PF4)
- net COL15: now reaches U1.40 (PF1)
- net COL16: now reaches U1.41 (PF0)
- net ENCODER: now reaches U1.42 (AREF)
- net ENCODER: now also C9.1, R7.2, R8.2, R9.1, SW2.S1
- net ROW5: now reaches U1.8 (PB0)
- net ROW4: now reaches U1.9 (PB1)
- new net: D111.2 (DOUT), D112.4 (DIN)
- new net: D110.2 (DOUT), D111.4 (DIN)
- new net: D110.4 (DIN), R6.1
- new net: R8.1, SW2.A
- new net: R7.1, SW2.B
- new net COL10: U1.22 (PD5)
- new net COL8: U1.20 (PD2)
- new net COL9: U1.19 (PD1)
Other:
- moved on the sheet: R2, R5
