File: metropolislefty.sch (KiCad schematic (older format))
At the start: 15 parts

Commit message: Created version 1.0 for fabrication
Parts:
- added C1: 4.7nF, Capacitor_SMD:C_0805_2012Metric, symbol Device:C_Small
- added C9: 10nF, Capacitor_SMD:C_0805_2012Metric, symbol Device:C_Small
- added D110, D111: WS2812B, LED_SMD:LED_WS2812B_PLCC4_5.0x5.0mm_P3.2mm, symbol LED:WS2812B
- added F1: 500mA, Fuse:Fuse_1206_3216Metric, symbol Device:Polyfuse_Small
- added R1: 1M, Resistor_SMD:R_0805_2012Metric, symbol Device:R_Small
- added R6: 300, Resistor_SMD:R_0805_2012Metric, symbol Device:R_Small
- added R7: 33K, Resistor_SMD:R_0805_2012Metric, symbol Device:R_Small
- added R8, R9: 15k, Resistor_SMD:R_0805_2012Metric, symbol Device:R_Small
- added SW2: Rotary_Encoder_Switch, Rotary_Encoder:RotaryEncoder_Alps_EC11E-Switch_Vertical_H20mm, symbol Device:Rotary_Encoder_Switch
- C2, C3, C4, C5, C6, C7, C8: renamed from C?; footprint (none) -> Capacitor_SMD:C_0805_2012Metric
- R2, R3, R4, R5: renamed from R?; footprint (none) -> Resistor_SMD:R_0805_2012Metric
- SW1: renamed from SW?; footprint (none) -> random-keyboard-parts:SKQG-1155865
- USB1: renamed from USB?; footprint (none) -> random-keyboard-parts:Molex-0548190589; symbol random-keyboard-parts:Molex-0548190589 -> metropolislefty-rescue:Molex-0548190589-random-keyboard-parts
- Y1: renamed from Y?; footprint (none) -> Crystal:Crystal_SMD_3225-4Pin_3.2x2.5mm
- gave numbers to parts that had none: 1
Connections:
- net labels added: ENCODER, STATUS_LEDS, VCC
- wire segments 59 -> 106
Other:
- moved on the sheet: C2, C3, C4, C5, C6, C7, C8, R2, R3, R4, R5, SW1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
