File: metropolislefty.sch (KiCad schematic (older format))
At the start: 26 parts, among them SW1 SW_Push, U1 ATmega32U4-AU, Y1 Crystal_GND24_Small

Commit message: Revision 1 Test w/ USB C
Parts:
- removed R1: 1M, Resistor_SMD:R_0805_2012Metric, symbol Device:R_Small
- removed USB1: Molex-0548190589, random-keyboard-parts:Molex-0548190589, symbol random-keyboard-parts:Molex-0548190589
- added D5, D6, D7: WS2812B, LED_SMD:LED_WS2812B_PLCC4_5.0x5.0mm_P3.2mm, symbol LED:WS2812B
- added R1, R6: 5k1, Resistor_SMD:R_0805_2012Metric, symbol Device:R
- added R10: 33k, Resistor_SMD:R_0805_2012Metric, symbol Device:R_Small
- added R7: 470, Resistor_SMD:R_0805_2012Metric, symbol Device:R_Small
- added R8, R9: 15k, Resistor_SMD:R_0805_2012Metric, symbol Device:R_Small
- added SW2: Rotary_Encoder_Switch, Rotary_Encoder:RotaryEncoder_Alps_EC11E-Switch_Vertical_H20mm, symbol Device:Rotary_Encoder_Switch
- added USB1: HRO-TYPE-C-31-M-12, Type-C:HRO-TYPE-C-31-M-12, symbol Type-C:HRO-TYPE-C-31-M-12
- C1: value 4.7nF -> 10nF
- D1, D2, D3, D4: footprint Diode_SMD:D_SOD-123 -> Diode_THT:D_DO-35_SOD27_P7.62mm_Horizontal
Connections:
- net +5V: now also D5.1 (VDD), D6.1 (VDD), D7.1 (VDD), R8.2
- net D+: now also USB1.6 (DP1), USB1.8 (DP2)
- net D-: now also USB1.5 (DN2), USB1.7 (DN1)
- net GND: now also D5.3 (VSS), D6.3 (VSS), D7.3 (VSS), R1.1, R6.2, SW2.C, SW2.S2, USB1.1 (GND), USB1.12 (GND), USB1.13 (SHIELD)
- net ROW0: now also U1.11 (PB3); no longer U1.19 (PD1)
- net VCC: now also USB1.11 (VBUS), USB1.2 (VBUS)
- net LEDS: now reaches U1.1 (PE6)
- net LEDS: now also R7.1
- net ENC: now reaches U1.42 (AREF)
- net ENC: now also C1.1, R10.1, R8.1, R9.1, SW2.S1
- new net: R6.1, USB1.10 (CC2)
- new net: R1.2, USB1.4 (CC1)
- new net: R9.2, SW2.A
- new net: R10.2, SW2.B
- new net: D5.2 (DOUT), D6.4 (DIN)
- new net: D5.4 (DIN), R7.2
- new net: D6.2 (DOUT), D7.4 (DIN)
Other:
- moved on the sheet: C2, C3, C4, C5, D1, D2, D3, D4, F1, MX1, MX2, MX3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
